Commit message: nyo

File: amir740_ros/amir_description/urdf/amir_mecanum3.gazebo.xacro (robot description, xacro)
@@ -39,8 +39,14 @@
             </plugin>
         </gazebo> -->
-        <gazebo>
+        <!-- <gazebo>
           <plugin filename="gz_ros2_control-system"
                   name="gz_ros2_control::GazeboSimROS2ControlPlugin">
             <parameters>$(find gz_ros2_control_demos)/config/cart_controller.yaml</parameters>
+          </plugin>
+        </gazebo> -->
+        <gazebo>
+          <plugin filename="ign_ros2_control-system"
+                  name="ign_ros2_control::IgnitionROS2ControlPlugin">
+            <parameters>$(find amir_bringup)/config/controllers.yaml</parameters>
           </plugin>
         </gazebo>

File: amir740_ros/amir_description/urdf/amir_mecanum3.gazebo_ros2_control.xacro (robot description, xacro)
@@ -15,5 +15,5 @@
         <state_interface name="effort"/>
       </joint>
-      <!-- <joint name="${name_joint_2}">
+      <joint name="${name_joint_2}">
         <command_interface name="position">
           <param name="min">${joint_2_lower_limit}</param>
@@ -85,5 +85,5 @@
       <state_interface name="velocity"/>
       <state_interface name="effort"/>
-    </joint> -->
+    </joint>
     </ros2_control>
   </xacro:macro>

File: amir740_ros/amir_description/urdf/amir_mecanum3.urdf (robot description, URDF)
Before this commit: robot amir_mecanum3, 21 links, 20 joints
Links:
- removed link back_lrf_link
- removed link front_lrf_link
Joints:
- removed joint back_lrf_joint
- removed joint front_lrf_joint
- joint base_joint: origin xyz=0 0 0 rpy=0 0 -1.5707963267948966 -> xyz=0 0 0 rpy=0 0 0

File: amir740_ros/amir_description/urdf/amir_mecanum3.xacro (robot description, xacro)
@@ -10,3 +10,48 @@
   <child link="link0_1"/>
 </joint>
+<!-- <xacro:include filename="$(find amir_description)/urdf/amir_mecanum3.gazebo.xacro"/>
+<xacro:include filename="$(find amir_description)/urdf/amir_mecanum3.gazebo_ros2_control.xacro"/>
+<xacro:gazebo_robot_settings />
+<xacro:amir_mecanum3_gazebo_ros2_control_settings name="AmirArmSystem" /> -->
+<ros2_control name="AmirRealHardware" type="system">
+    <hardware>
+      <plugin>amir_driver/AmirHardwareInterfaces</plugin>
+    </hardware>
+    <joint name="Joint_1">
+      <command_interface name="position"/>
+      <command_interface name="velocity"/>
+      <state_interface name="position"/>
+      <state_interface name="velocity"/>
+    </joint>
+    <joint name="Joint_2">
+      <command_interface name="position"/>
+      <command_interface name="velocity"/>
+      <state_interface name="position"/>
+      <state_interface name="velocity"/>
+    </joint>
+    <joint name="Joint_3">
+      <command_interface name="position"/>
+      <command_interface name="velocity"/>
+      <state_interface name="position"/>
+      <state_interface name="velocity"/>
+    </joint>
+    <joint name="Joint_4">
+      <command_interface name="position"/>
+      <command_interface name="velocity"/>
+      <state_interface name="position"/>
+      <state_interface name="velocity"/>
+    </joint>
+    <joint name="Joint_5">
+      <command_interface name="position"/>
+      <command_interface name="velocity"/>
+      <state_interface name="position"/>
+      <state_interface name="velocity"/>
+    </joint>
+    <joint name="Gripper">
+      <command_interface name="position"/>
+      <command_interface name="velocity"/>
+      <state_interface name="position"/>
+      <state_interface name="velocity"/>
+    </joint>
+  </ros2_control>
 </robot>

File: amir740_ros/amir_moveit_config/config/amir_mecanum3.ros2_control.xacro (robot description, xacro)
@@ -1,7 +1,7 @@
 <?xml version="1.0"?>
 <robot xmlns:xacro="http://www.ros.org/wiki/xacro">
-    <xacro:macro name="amir_ros2_control" params="ros2_control_hardware_type">
-        <!-- <xacro:property name="initial_positions" value="${xacro.load_yaml(initial_positions_file)['initial_positions']}"/> -->
-        <ros2_control name="amir_ros2" type="system">
+    <xacro:macro name="amir_mecanum3_ros2_control" params="name initial_positions_file ros2_control_hardware_type">
+        <xacro:property name="initial_positions" value="${load_yaml(initial_positions_file)['initial_positions']}"/>
+        <ros2_control name="${name}" type="system">
             <hardware>
                 <xacro:if value="${ros2_control_hardware_type == 'mock_components'}">
@@ -12,9 +12,12 @@
                 </xacro:if>
             </hardware>
+        <!-- <ros2_control name="${name}" type="system">
+            <hardware>
+                <plugin>mock_components/GenericSystem</plugin>
+            </hardware> -->
             <joint name="Joint_1">
                 <command_interface name="position"/>
-                <command_interface name="velocity"/>
                 <state_interface name="position">
-                  <!-- <param name="initial_value">0.0</param> -->
+                  <param name="initial_value">${initial_positions['Joint_1']}</param>
                 </state_interface>
                 <state_interface name="velocity"/>
@@ -22,7 +25,6 @@
             <joint name="Joint_2">
                 <command_interface name="position"/>
-                <command_interface name="velocity"/>
                 <state_interface name="position">
-                  <!-- <param name="initial_value">0.0</param> -->
+                  <param name="initial_value">${initial_positions['Joint_2']}</param>
                 </state_interface>
                 <state_interface name="velocity"/>
@@ -30,7 +32,6 @@
             <joint name="Joint_3">
                 <command_interface name="position"/>
-                <command_interface name="velocity"/>
                 <state_interface name="position">
-                  <!-- <param name="initial_value">0.0</param> -->
+                  <param name="initial_value">${initial_positions['Joint_3']}</param>
                 </state_interface>
                 <state_interface name="velocity"/>
@@ -38,7 +39,6 @@
             <joint name="Joint_4">
                 <command_interface name="position"/>
-                <command_interface name="velocity"/>
                 <state_interface name="position">
-                  <!-- <param name="initial_value">0.0</param> -->
+                  <param name="initial_value">${initial_positions['Joint_4']}</param>
                 </state_interface>
                 <state_interface name="velocity"/>
@@ -46,7 +46,6 @@
             <joint name="Joint_5">
                 <command_interface name="position"/>
-                <command_interface name="velocity"/>
                 <state_interface name="position">
-                  <!-- <param name="initial_value">0.0</param> -->
+                  <param name="initial_value">${initial_positions['Joint_5']}</param>
                 </state_interface>
                 <state_interface name="velocity"/>
@@ -55,7 +54,7 @@
                 <command_interface name="position"/>
                 <state_interface name="position">
-                  <!-- <param name="initial_value">0.0</param> -->
+                  <param name="initial_value">${initial_positions['Gripper']}</param>
                 </state_interface>
-                <!-- <state_interface name="velocity"/> -->
+                <state_interface name="velocity"/>
             </joint>
         </ros2_control>

File: amir740_ros/new_amir_description/urdf/mecanum3.xacro (robot description, xacro)
@@ -10,5 +10,6 @@
   <parent link="base_footprint"/>
   <child link="base_link" />
-  <origin xyz="0 0 0" rpy="0 0 ${radians(-90)}"/>
+  <!-- <origin xyz="0 0 0" rpy="0 0 ${radians(-90)}"/> -->
+  <origin xyz="0 0 0" rpy="0 0 0"/>
 </joint>
 <link name="base_link">

File: amir740_ros/new_amir_description/urdf/旧new_amir.urdf (robot description, URDF)
Before this commit: robot amir_mecanum3, 19 links, 18 joints
Joints:
- joint base_joint: origin xyz=0 0 0 rpy=0 0 0 -> xyz=0 0 0 rpy=0 0 -1.5707963267948966
