Commit message: gaeboバージョン更新、nav2少し

File: amir740_ros/amir_description/urdf/amir_mecanum3_sim.xacro (robot description, xacro)
@@ -2,8 +2,8 @@
 <robot name="amir_mecanum3" xmlns:xacro="http://www.ros.org/wiki/xacro">
   <!-- メカナムローバー URDF
-       mecanum3.gazebo (libgazebo_ros2_control.so) と
+       mecanum3.gazebo (gz_ros2_control-system) と
        mecanum3_ros2_control.xacro (MecanumSystem) を含む -->
   <xacro:include filename="$(find mecanumrover_description)/urdf/mecanum3.xacro"/>
-  <!-- AMIR アーム リンク/ジョイント (gazebo インクルードはコメントアウト済み) -->
+  <!-- AMIR アーム リンク/ジョイント -->
   <xacro:include filename="$(find amir_description)/urdf/amir_for_rover.xacro"/>
   <!-- ローバーとアームの固定接続 -->
@@ -13,10 +13,10 @@
     <child link="link0_1"/>
   </joint>
-  <!-- AMIR アーム Gazebo シミュレーション用 ros2_control
-       libgazebo_ros2_control.so は URDF 内の全 <ros2_control> タグを読み込み
-       GazeboSystem としてシミュレーションする -->
+  <!-- AMIR アーム Ignition Gazebo 用 ros2_control
+       gz_ros2_control-system プラグインが URDF 内の全 <ros2_control> タグを
+       読み込み GazeboSimSystem としてシミュレーションする -->
   <ros2_control name="AmirGazeboSystem" type="system">
     <hardware>
-      <plugin>gazebo_ros2_control/GazeboSystem</plugin>
+      <plugin>gz_ros2_control/GazeboSimSystem</plugin>
     </hardware>
     <joint name="Joint_1">
@@ -116,73 +116,77 @@
     </joint>
   </ros2_control>
-  <!-- AMIR アームリンクの Gazebo マテリアル設定 -->
-  <gazebo reference="link0_1">
-    <material>Gazebo/Silver</material>
-    <mu1>1.4</mu1><mu2>1.4</mu2>
-    <selfCollide>true</selfCollide>
-  </gazebo>
-  <gazebo reference="link1_1">
-    <material>Gazebo/Silver</material>
-    <mu1>1.4</mu1><mu2>1.4</mu2>
-    <selfCollide>true</selfCollide>
-  </gazebo>
-  <gazebo reference="link2_1">
-    <material>Gazebo/Silver</material>
-    <mu1>1.4</mu1><mu2>1.4</mu2>
-    <selfCollide>true</selfCollide>
-  </gazebo>
-  <gazebo reference="link3_1">
-    <material>Gazebo/Silver</material>
-    <mu1>1.4</mu1><mu2>1.4</mu2>
-    <selfCollide>true</selfCollide>
-  </gazebo>
-  <gazebo reference="link4_1">
-    <material>Gazebo/Silver</material>
-    <mu1>1.4</mu1><mu2>1.4</mu2>
-    <selfCollide>true</selfCollide>
-  </gazebo>
-  <gazebo reference="gripper_base_1">
-    <material>Gazebo/Silver</material>
-    <mu1>1.4</mu1><mu2>1.4</mu2>
-    <selfCollide>true</selfCollide>
-  </gazebo>
-  <gazebo reference="inner_link_left_1">
-    <material>Gazebo/Silver</material>
-    <mu1>2.0</mu1><mu2>2.0</mu2>
-    <selfCollide>false</selfCollide>
-  </gazebo>
-  <gazebo reference="inner_link_right_1">
-    <material>Gazebo/Silver</material>
-    <mu1>2.0</mu1><mu2>2.0</mu2>
-    <selfCollide>false</selfCollide>
-  </gazebo>
-  <gazebo reference="outer_link_left_1">
-    <material>Gazebo/Silver</material>
-    <mu1>2.0</mu1><mu2>2.0</mu2>
-    <selfCollide>false</selfCollide>
-  </gazebo>
-  <gazebo reference="outer_link_right_1">
-    <material>Gazebo/Silver</material>
-    <mu1>2.0</mu1><mu2>2.0</mu2>
-    <selfCollide>false</selfCollide>
-  </gazebo>
-  <!-- finger_left/right_1: 把持面なので高摩擦 + 接触剛性を設定 -->
-  <!-- finger_left/right_1: 把持面なので高摩擦 + 接触剛性を設定
-       kp=1e6: すり抜け防止に必要な硬さ
-       kd=1e3: 接触振動を減衰 (旧値 1e2 → 10倍) -->
+  <!-- AMIR アームリンクの Ignition Gazebo 摩擦設定
+       Classic Gazebo: <mu1>/<mu2>/<kp>/<kd> を <gazebo reference> 直下に記述
+       Ignition Gazebo: <collision><surface><friction><ode> 階層が必要 -->
+  <gazebo reference="link0_1"><collision><surface><friction><ode>
+    <mu>1.4</mu><mu2>1.4</mu2>
+  </ode></friction></surface></collision></gazebo>
+  <gazebo reference="link1_1"><collision><surface><friction><ode>
+    <mu>1.4</mu><mu2>1.4</mu2>
+  </ode></friction></surface></collision></gazebo>
+  <gazebo reference="link2_1"><collision><surface><friction><ode>
+    <mu>1.4</mu><mu2>1.4</mu2>
+  </ode></friction></surface></collision></gazebo>
+  <gazebo reference="link3_1"><collision><surface><friction><ode>
+    <mu>1.4</mu><mu2>1.4</mu2>
+  </ode></friction></surface></collision></gazebo>
+  <gazebo reference="link4_1"><collision><surface><friction><ode>
+    <mu>1.4</mu><mu2>1.4</mu2>
+  </ode></friction></surface></collision></gazebo>
+  <gazebo reference="gripper_base_1"><collision><surface><friction><ode>
+    <mu>1.4</mu><mu2>1.4</mu2>
+  </ode></friction></surface></collision></gazebo>
+  <gazebo reference="inner_link_left_1"><collision><surface><friction><ode>
+    <mu>2.0</mu><mu2>2.0</mu2>
+  </ode></friction></surface></collision></gazebo>
+  <gazebo reference="inner_link_right_1"><collision><surface><friction><ode>
+    <mu>2.0</mu><mu2>2.0</mu2>
+  </ode></friction></surface></collision></gazebo>
+  <gazebo reference="outer_link_left_1"><collision><surface><friction><ode>
+    <mu>2.0</mu><mu2>2.0</mu2>
+  </ode></friction></surface></collision></gazebo>
+  <gazebo reference="outer_link_right_1"><collision><surface><friction><ode>
+    <mu>2.0</mu><mu2>2.0</mu2>
+  </ode></friction></surface></collision></gazebo>
+  <!-- グリッパー指: 高摩擦 + 接触剛性 (把持面) -->
   <gazebo reference="finger_left_1">
-    <material>Gazebo/Silver</material>
-    <mu1>3.0</mu1><mu2>3.0</mu2>
-    <kp>1e6</kp><kd>1e3</kd>
-    <selfCollide>false</selfCollide>
+    <collision>
+      <surface>
+        <friction>
+          <ode>
+            <mu>3.0</mu>
+            <mu2>3.0</mu2>
+          </ode>
+        </friction>
+        <contact>
+          <ode>
+            <kp>1e6</kp>
+            <kd>1e3</kd>
+            <max_vel>0.01</max_vel>
+            <min_depth>0.001</min_depth>
+          </ode>
+        </contact>
+      </surface>
+    </collision>
   </gazebo>
   <gazebo reference="finger_right_1">
-    <material>Gazebo/Silver</material>
-    <mu1>3.0</mu1><mu2>3.0</mu2>
-    <kp>1e6</kp><kd>1e3</kd>
-    <selfCollide>false</selfCollide>
-  </gazebo>
-  <gazebo reference="tcp_link">
-    <material>Gazebo/RedTransparent</material>
+    <collision>
+      <surface>
+        <friction>
+          <ode>
+            <mu>3.0</mu>
+            <mu2>3.0</mu2>
+          </ode>
+        </friction>
+        <contact>
+          <ode>
+            <kp>1e6</kp>
+            <kd>1e3</kd>
+            <max_vel>0.01</max_vel>
+            <min_depth>0.001</min_depth>
+          </ode>
+        </contact>
+      </surface>
+    </collision>
   </gazebo>
 </robot>

File: mecanumrover3_ros2/mecanumrover_description/urdf/mecanum3.xacro (robot description, xacro)
@@ -4,4 +4,5 @@
   <xacro:include filename="$(find mecanumrover_description)/urdf/mecanum3.gazebo" />
   <xacro:include filename="$(find mecanumrover_description)/urdf/mecanum3_ros2_control.xacro" />
+  <xacro:include filename="$(find vs_rover_options_description)/urdf/lrf/tg30_mecanum3.xacro" />
   <!-- Arm link macro -->
   <xacro:macro name="mecanum_arm_link" params="name">

File: mecanumrover3_ros2/mecanumrover_description/urdf/mecanum3_ros2_control.xacro (robot description, xacro)
@@ -3,23 +3,39 @@
   <ros2_control name="MecanumSystem" type="system">
     <hardware>
-      <plugin>gazebo_ros2_control/GazeboSystem</plugin>
+      <!-- Ignition Gazebo hardware plugin (replaces gazebo_ros2_control/GazeboSystem) -->
+      <plugin>gz_ros2_control/GazeboSimSystem</plugin>
     </hardware>
-    <!-- Wheel joints: STATE interfaces only (no command interface).
-         libgazebo_ros_diff_drive.so controls these joints directly via the Gazebo
-         physics API. If a velocity command_interface were present here, GazeboSystem
-         would initialise it to 0 and fight the diff_drive plugin. -->
+    <!-- Wheel joints: velocity COMMAND interfaces required by mecanum_drive_controller.
+         Classic Gazebo used libgazebo_ros_diff_drive.so which bypassed ros2_control.
+         In Ignition, mecanum_drive_controller drives the wheels via these interfaces. -->
     <joint name="front_left_joint">
+      <command_interface name="velocity">
+        <param name="min">-20.0</param>
+        <param name="max">20.0</param>
+      </command_interface>
       <state_interface name="position"/>
       <state_interface name="velocity"/>
     </joint>
     <joint name="front_right_joint">
+      <command_interface name="velocity">
+        <param name="min">-20.0</param>
+        <param name="max">20.0</param>
+      </command_interface>
       <state_interface name="position"/>
       <state_interface name="velocity"/>
     </joint>
     <joint name="back_left_joint">
+      <command_interface name="velocity">
+        <param name="min">-20.0</param>
+        <param name="max">20.0</param>
+      </command_interface>
       <state_interface name="position"/>
       <state_interface name="velocity"/>
     </joint>
     <joint name="back_right_joint">
+      <command_interface name="velocity">
+        <param name="min">-20.0</param>
+        <param name="max">20.0</param>
+      </command_interface>
       <state_interface name="position"/>
       <state_interface name="velocity"/>
