Commit message: namespace,multirobot

File: amir740_ros/amir_description/urdf/amir_mecanum3_sim.xacro (robot description, xacro)
@@ -1,4 +1,9 @@
 <?xml version="1.0" ?>
 <robot name="amir_mecanum3" xmlns:xacro="http://www.ros.org/wiki/xacro">
+  <!-- マルチロボット用 namespace 引数 (空なら従来どおり単体・無 prefix)
+       include 先 (mecanum3.gazebo / tg30_mecanum3.gazebo / _d435.gazebo.xacro)
+       が Ignition 側の topic / frame_id を ${namespace}/ で prefix する。
+       TF フレーム自体は launch 側 robot_state_publisher の frame_prefix で付与。 -->
+  <xacro:arg name="namespace" default=""/>
   <!-- メカナムローバー URDF
        mecanum3.gazebo (gz_ros2_control-system) と

File: vs_rover_options_description/urdf/depth_cam/_d435.gazebo.xacro (robot description, xacro)
@@ -9,4 +9,8 @@
 -->
 <robot xmlns:xacro="http://ros.org/wiki/xacro">
+  <!-- マルチロボット用 namespace (空なら従来どおり無 prefix) -->
+  <xacro:arg name="namespace" default=""/>
+  <xacro:property name="robot_ns" value="$(arg namespace)"/>
+  <xacro:property name="ns_prefix" value="${robot_ns + '/' if robot_ns else ''}"/>
   <xacro:macro name="gazebo_d435" params="camera_name reference_link topics_ns depth_optical_frame color_optical_frame infrared1_optical_frame infrared2_optical_frame publish_pointcloud:=true">
     <gazebo reference="${reference_link}">
@@ -38,5 +42,5 @@
         <update_rate>5</update_rate>
         <visualize>true</visualize>
-        <topic>${topics_ns}</topic>
+        <topic>/${ns_prefix}${topics_ns}</topic>
         <ignition_frame_id>${depth_optical_frame}</ignition_frame_id>
       </sensor>
