Commit message: sim

File: amir740_ros/amir_description/urdf/amir_for_rover.xacro (robot description, xacro)
@@ -4,6 +4,6 @@
 <xacro:include filename="$(find amir_description)/urdf/amir.trans" />
 <!-- <xacro:include filename="$(find amir_description)/urdf/amir.gazebo" />新しいros2用のやつを作る -->
-<xacro:include filename="$(find amir_description)/urdf/amir_mecanum3.gazebo.xacro" />
-<xacro:include filename="$(find amir_description)/urdf/amir_mecanum3.gazebo_ros2_control.xacro" />
+<!-- <xacro:include filename="$(find amir_description)/urdf/amir_mecanum3.gazebo.xacro" />
+<xacro:include filename="$(find amir_description)/urdf/amir_mecanum3.gazebo_ros2_control.xacro" /> -->
 <link name="link0_1">
   <inertial>
@@ -424,43 +424,48 @@
   <limit lower="-1.047198" upper="0.261799" effort="0.4" velocity="2"/>
 </joint>
-<joint name="left_inner_back_joint" type="continuous">
+<joint name="left_inner_back_joint" type="revolute">
   <origin xyz="-0.017633 0.020522 0.0" rpy="0 0 0"/>
   <parent link="gripper_base_1"/>
   <child link="inner_link_left_1"/>
   <axis xyz="0.0 0.0 -1.0"/>
-  <!-- <limit lower="-1.047198" upper="0.261799" effort="10" velocity="4"/> -->
-  <mimic joint="Gripper" multiplier="1" offset="0" />
-</joint>
-<joint name="right_outer_back_joint" type="continuous">
+  <limit lower="-1.047198" upper="0.261799" effort="0.4" velocity="2"/>
+  <dynamics damping="0.1" friction="0.05"/>
+  <mimic joint="Gripper" multiplier="1" offset="0" />
+</joint>
+<joint name="right_outer_back_joint" type="revolute">
   <origin xyz="0.038367 0.020522 0.0" rpy="0 0 0"/>
   <parent link="gripper_base_1"/>
   <child link="outer_link_right_1"/>
   <axis xyz="0.0 0.0 1.0"/>
-  <!-- <limit lower="-1.047198" upper="0.261799" effort="10" velocity="4"/> -->
-  <mimic joint="Gripper" multiplier="1" offset="0" />
-</joint>
-<joint name="left_outer_back_joint" type="continuous">
+  <limit lower="-1.047198" upper="0.261799" effort="0.4" velocity="2"/>
+  <dynamics damping="0.1" friction="0.05"/>
+  <mimic joint="Gripper" multiplier="1" offset="0" />
+</joint>
+<joint name="left_outer_back_joint" type="revolute">
   <origin xyz="-0.037633 0.020522 0.0" rpy="0 0 0"/>
   <parent link="gripper_base_1"/>
   <child link="outer_link_left_1"/>
   <axis xyz="0.0 0.0 -1.0"/>
-  <!-- <limit lower="-1.047198" upper="0.261799" effort="10" velocity="4"/> -->
+  <limit lower="-1.047198" upper="0.261799" effort="0.4" velocity="2"/>
+  <dynamics damping="0.1" friction="0.05"/>
   <mimic joint="Gripper" multiplier="1" offset="0" />
 </joint>
 <!-- use this when using inner joint -->
-<joint name="right_inner_front_joint" type="continuous">
+<joint name="right_inner_front_joint" type="revolute">
   <origin xyz="0.0 0.04 0.0" rpy="0 0 0"/>
   <parent link="inner_link_right_1"/>
   <child link="finger_right_1"/>
   <axis xyz="0.0 0.0 -1.0"/>
-  <!-- <limit lower="-1.047198" upper="0.261799" effort="10" velocity="4"/> -->
-  <mimic joint="Gripper" multiplier="1" offset="0" />
-</joint>
-<joint name="left_inner_front_joint" type="continuous">
+  <limit lower="-1.047198" upper="0.261799" effort="0.4" velocity="2"/>
+  <dynamics damping="0.1" friction="0.05"/>
+  <mimic joint="Gripper" multiplier="1" offset="0" />
+</joint>
+<joint name="left_inner_front_joint" type="revolute">
   <origin xyz="-0.0 0.04 0.0" rpy="0 0 0"/>
   <parent link="inner_link_left_1"/>
   <child link="finger_left_1"/>
   <axis xyz="0.0 0.0 1.0"/>
-  <!-- <limit lower="-1.047198" upper="0.261799" effort="10" velocity="4"/> -->
+  <limit lower="-1.047198" upper="0.261799" effort="0.4" velocity="2"/>
+  <dynamics damping="0.1" friction="0.05"/>
   <mimic joint="Gripper" multiplier="1" offset="0" />
 </joint>

Commit message: gazebo修正

File: amir740_ros/amir_description/urdf/amir_for_rover.xacro (robot description, xacro)
@@ -383,5 +383,6 @@
   <axis xyz="0.0 0.0 1.0"/>
   <limit upper="2.96706" lower="-2.96706" effort="33" velocity="1"/>
-  <dynamics damping="0.6" friction="0.3" />
+  <!-- Increased damping to reduce arm reaction forces transmitted to the mobile base -->
+  <dynamics damping="3.0" friction="0.3" />
 </joint>
 <joint name="Joint_2" type="revolute">
@@ -391,5 +392,5 @@
   <axis xyz="1.0 0.0 0.0"/>
   <limit upper="2.356194" lower="0" effort="22" velocity="1"/>
-  <dynamics damping="0.6" friction="0.3" />
+  <dynamics damping="3.0" friction="0.3" />
 </joint>
 <joint name="Joint_3" type="revolute">
@@ -399,5 +400,5 @@
   <axis xyz="1.0 0.0 0.0"/>
   <limit upper="0.0" lower="-2.792527" effort="26" velocity="1"/>
-  <dynamics damping="0.6" friction="0.3" />
+  <dynamics damping="3.0" friction="0.3" />
 </joint>
 <joint name="Joint_4" type="revolute">
@@ -407,5 +408,5 @@
   <axis xyz="1.0 0.0 0.0"/>
   <limit lower="-2.094395" upper="1.308997" effort="1.3" velocity="1"/>
-  <dynamics damping="0.3" friction="0.1" />
+  <dynamics damping="1.5" friction="0.1" />
 </joint>
 <joint name="Joint_5" type="revolute">
@@ -415,5 +416,5 @@
   <axis xyz="0.0 1.0 0.0"/>
   <limit lower="-2.75762" upper="2.75762" effort="0.4" velocity="2"/>
-  <dynamics damping="0.3" friction="0.1" />
+  <dynamics damping="1.5" friction="0.1" />
 </joint>
 <joint name="Gripper" type="revolute">

File: mecanumrover3_ros2/mecanumrover_description/urdf/mecanum3.xacro (robot description, xacro)
@@ -4,97 +4,4 @@
   <xacro:include filename="$(find mecanumrover_description)/urdf/mecanum3.gazebo" />
   <xacro:include filename="$(find mecanumrover_description)/urdf/mecanum3_ros2_control.xacro" />
-  <!-- OPTION LRF TG30 -->
-  <!-- <xacro:include filename="$(find vs_rover_options_description)/urdf/lrf/tg30_mecanum3.xacro" /> -->
-  <!-- Inertial macros -->
-  <xacro:macro name="cylinder_inertial" params="mass radius length">
-    <mass value="${mass}"/>
-    <inertia
-      ixx="${((radius*radius)/4 + (length*length)/12)*mass}"
-      ixy="0" ixz="0"
-      iyy="${((radius*radius)/4 + (length*length)/12)*mass}"
-      iyz="0"
-      izz="${(mass*radius*radius)/2}" />
-  </xacro:macro>
-  <!-- Barrel (roller) macros  -->
-  <xacro:macro name="barrel_rl" params="prefix parent dir rot">
-    <joint name="${prefix}_joint" type="continuous">
-      <parent link="${parent}"/>
-      <child  link="${prefix}_link"/>
-      <origin
-        xyz="${0.0666389*cos(radians(dir))} ${0.0666389*sin(radians(dir))} 0"
-        rpy="${pi/4*rot} 0 ${radians(dir)}"/>
-      <axis xyz="0 0 1"/>
-      <dynamics damping="0.001" friction="0.001"/>
-    </joint>
-    <link name="${prefix}_link">
-      <visual>
-        <geometry>
-          <mesh filename="package://mecanumrover_description/meshes/mecanum3/mecanum_barrel.stl"/>
-        </geometry>
-        <material name="dark_grey"/>
-      </visual>
-      <collision>
-        <geometry>
-          <mesh filename="package://mecanumrover_description/meshes/mecanum3/mecanum_barrel.stl"/>
-        </geometry>
-      </collision>
-      <inertial>
-        <xacro:cylinder_inertial
-          mass="0.01225"
-          radius="0.00956"
-          length="0.0381"/>
-      </inertial>
-    </link>
-  </xacro:macro>
-  <xacro:macro name="barrels_rl" params="prefix parent rot">
-    <xacro:barrel_rl prefix="${prefix}_0"  parent="${parent}" dir="0"   rot="${rot}"/>
-    <xacro:barrel_rl prefix="${prefix}_1"  parent="${parent}" dir="24"  rot="${rot}"/>
-    <xacro:barrel_rl prefix="${prefix}_2"  parent="${parent}" dir="48"  rot="${rot}"/>
-    <xacro:barrel_rl prefix="${prefix}_3"  parent="${parent}" dir="72"  rot="${rot}"/>
-    <xacro:barrel_rl prefix="${prefix}_4"  parent="${parent}" dir="96"  rot="${rot}"/>
-    <xacro:barrel_rl prefix="${prefix}_5"  parent="${parent}" dir="120" rot="${rot}"/>
-    <xacro:barrel_rl prefix="${prefix}_6"  parent="${parent}" dir="144" rot="${rot}"/>
-    <xacro:barrel_rl prefix="${prefix}_7"  parent="${parent}" dir="168" rot="${rot}"/>
-    <xacro:barrel_rl prefix="${prefix}_8"  parent="${parent}" dir="192" rot="${rot}"/>
-    <xacro:barrel_rl prefix="${prefix}_9"  parent="${parent}" dir="216" rot="${rot}"/>
-    <xacro:barrel_rl prefix="${prefix}_10" parent="${parent}" dir="240" rot="${rot}"/>
-    <xacro:barrel_rl prefix="${prefix}_11" parent="${parent}" dir="264" rot="${rot}"/>
-    <xacro:barrel_rl prefix="${prefix}_12" parent="${parent}" dir="288" rot="${rot}"/>
-    <xacro:barrel_rl prefix="${prefix}_13" parent="${parent}" dir="312" rot="${rot}"/>
-    <xacro:barrel_rl prefix="${prefix}_14" parent="${parent}" dir="336" rot="${rot}"/>
-  </xacro:macro>
-  <xacro:macro name="attach_mecanum_rollers" params="wheel_prefix wheel_link rot">
-    <xacro:barrels_rl
-      prefix="${wheel_prefix}_barrel"
-      parent="${wheel_link}"
-      rot="${rot}"/>
-  </xacro:macro>
-  <!-- Base -->
-  <link name="base_footprint"/>
-  <joint name="base_joint" type="fixed">
-    <parent link="base_footprint"/>
-    <child link="base_link"/>
-    <origin xyz="0 0 0" rpy="0 0 -1.5708"/>
-  </joint>
-  <link name="base_link">
-    <inertial>
-      <origin xyz="0.000129 -0.001817 0.110883"/>
-      <mass value="40"/>
-      <inertia ixx="1.346868e-01" iyy="4.468661e-02" izz="1.499091e-01" ixy="3.076527e-04" ixz="-2.931603e-05" iyz="2.763693e-05"/>
-    </inertial>
-    <visual>
-      <geometry>
-        <mesh filename="package://mecanumrover_description/meshes/mecanum3/base_link.stl"
-              scale="0.001 0.001 0.001"/>
-      </geometry>
-      <material name="silver"/>
-    </visual>
-    <collision>
-      <geometry>
-        <mesh filename="package://mecanumrover_description/meshes/mecanum3/base_link.stl"
-              scale="0.001 0.001 0.001"/>
-      </geometry>
-    </collision>
-  </link>
   <!-- Arm link macro -->
   <xacro:macro name="mecanum_arm_link" params="name">
@@ -120,17 +27,7 @@
     </link>
   </xacro:macro>
-  <!-- Suspension joint macro -->
-  <xacro:macro name="mecanum_suspension_joint"
-               params="name parent child xyz rpy">
-    <joint name="${name}" type="revolute">
-      <parent link="${parent}"/>
-      <child link="${child}"/>
-      <origin xyz="${xyz}" rpy="${rpy}"/>
-      <axis xyz="1 0 0"/>
-      <limit lower="-0.10472" upper="0" effort="300" velocity="20"/>
-      <dynamics damping="5.0" friction="0.1"/>
-    </joint>
-  </xacro:macro>
-  <!-- Wheel link macros -->
+  <!-- Wheel link macros
+       Collision changed from mecanum STL mesh to cylinder for stable ODE contact.
+       radius=0.076 matches the mecanum outer radius (barrel center 0.0666 + barrel radius 0.00956). -->
   <xacro:macro name="mecanum_wheel_link" params="name">
     <link name="${name}">
@@ -149,6 +46,5 @@
       <collision>
         <geometry>
-          <mesh filename="package://mecanumrover_description/meshes/mecanum3/mecanum_wheel.stl"
-                scale="0.001 0.001 0.001"/>
+          <cylinder radius="0.076" length="0.05"/>
         </geometry>
       </collision>
@@ -171,6 +67,5 @@
       <collision>
         <geometry>
-          <mesh filename="package://mecanumrover_description/meshes/mecanum3/mecanum_wheel_rev.stl"
-                scale="0.001 0.001 0.001"/>
+          <cylinder radius="0.076" length="0.05"/>
         </geometry>
       </collision>
@@ -178,6 +73,5 @@
   </xacro:macro>
   <!-- Wheel joint macro -->
-  <xacro:macro name="mecanum_wheel_joint"
-               params="name parent child xyz rpy axis_z">
+  <xacro:macro name="mecanum_wheel_joint" params="name parent child xyz rpy axis_z">
     <joint name="${name}" type="continuous">
       <parent link="${parent}"/>
@@ -185,11 +79,35 @@
       <origin xyz="${xyz}" rpy="${rpy}"/>
       <axis xyz="0 0 ${axis_z}"/>
-      <!-- effort limit is required: GazeboSystem uses it as ODE fmax.
-           Without it fmax=0 and the velocity controller applies zero torque,
-           letting reaction forces from the arm push the base freely. -->
-      <limit effort="1500.0" velocity="20.0"/>
-      <dynamics damping="1.0" friction="0.0"/>
+      <limit effort="2500.0" velocity="20.0"/>
+      <dynamics damping="0.1" friction="0.0"/>
     </joint>
   </xacro:macro>
+  <!-- Base -->
+  <link name="base_footprint"/>
+  <joint name="base_joint" type="fixed">
+    <parent link="base_footprint"/>
+    <child link="base_link"/>
+    <origin xyz="0 0 0" rpy="0 0 -1.5708"/>
+  </joint>
+  <link name="base_link">
+    <inertial>
+      <origin xyz="0.000129 -0.001817 0.110883"/>
+      <mass value="20"/>
+      <inertia ixx="1.346868e-01" iyy="4.468661e-02" izz="1.499091e-01" ixy="3.076527e-04" ixz="-2.931603e-05" iyz="2.763693e-05"/>
+    </inertial>
+    <visual>
+      <geometry>
+        <mesh filename="package://mecanumrover_description/meshes/mecanum3/base_link.stl"
+              scale="0.001 0.001 0.001"/>
+      </geometry>
+      <material name="silver"/>
+    </visual>
+    <collision>
+      <geometry>
+        <mesh filename="package://mecanumrover_description/meshes/mecanum3/base_link.stl"
+              scale="0.001 0.001 0.001"/>
+      </geometry>
+    </collision>
+  </link>
   <!-- Arms -->
   <xacro:mecanum_arm_link name="front_left_arm"/>
@@ -197,29 +115,25 @@
   <xacro:mecanum_arm_link name="back_left_arm"/>
   <xacro:mecanum_arm_link name="back_right_arm"/>
-  <!-- Suspension joints -->
-  <xacro:mecanum_suspension_joint
-    name="front_left_suspension_joint"
-    parent="base_link"
-    child="front_left_arm"
-    xyz="-0.085 0.020 0.076"
-    rpy="0 0 ${radians(180)}"/>
-  <xacro:mecanum_suspension_joint
-    name="front_right_suspension_joint"
-    parent="base_link"
-    child="front_right_arm"
-    xyz="0.085 0.020 0.076"
-    rpy="0 0 ${radians(180)}"/>
-  <xacro:mecanum_suspension_joint
-    name="back_left_suspension_joint"
-    parent="base_link"
-    child="back_left_arm"
-    xyz="-0.085 -0.020 0.076"
-    rpy="0 0 0"/>
-  <xacro:mecanum_suspension_joint
-    name="back_right_suspension_joint"
-    parent="base_link"
-    child="back_right_arm"
-    xyz="0.085 -0.020 0.076"
-    rpy="0 0 0"/>
+  <!-- Suspension joints (fixed: eliminates oscillation that caused tipping) -->
+  <joint name="front_left_suspension_joint" type="fixed">
+    <parent link="base_link"/>
+    <child link="front_left_arm"/>
+    <origin xyz="-0.085 0.020 0.076" rpy="0 0 ${radians(180)}"/>
+  </joint>
+  <joint name="front_right_suspension_joint" type="fixed">
+    <parent link="base_link"/>
+    <child link="front_right_arm"/>
+    <origin xyz="0.085 0.020 0.076" rpy="0 0 ${radians(180)}"/>
+  </joint>
+  <joint name="back_left_suspension_joint" type="fixed">
+    <parent link="base_link"/>
+    <child link="back_left_arm"/>
+    <origin xyz="-0.085 -0.020 0.076" rpy="0 0 0"/>
+  </joint>
+  <joint name="back_right_suspension_joint" type="fixed">
+    <parent link="base_link"/>
+    <child link="back_right_arm"/>
+    <origin xyz="0.085 -0.020 0.076" rpy="0 0 0"/>
+  </joint>
   <!-- Wheels -->
   <xacro:mecanum_wheel_rev_link name="front_left_wheel_1"/>
@@ -227,5 +141,8 @@
   <xacro:mecanum_wheel_link     name="back_left_wheel_1"/>
   <xacro:mecanum_wheel_rev_link name="back_right_wheel_1"/>
-  <!-- Wheel joints -->
+  <!-- Wheel joints
+       axis_z signs corrected so that +velocity → robot moves in +X (forward in base_footprint).
+       base_joint is rotated Rz(-90°), making all wheel axes land on -Y in base_footprint
+       with the original signs; negating them flips to +Y which gives forward motion. -->
   <xacro:mecanum_wheel_joint
     name="front_left_joint"
@@ -234,5 +151,5 @@
     xyz="0.03 -0.100 0"
     rpy="0 ${radians(-270)} 0"
-    axis_z="-1"/>
+    axis_z="1"/>
   <xacro:mecanum_wheel_joint
     name="front_right_joint"
@@ -241,5 +158,5 @@
     xyz="-0.03 -0.100 0"
     rpy="0 ${radians(-90)} 0"
-    axis_z="1"/>
+    axis_z="-1"/>
   <xacro:mecanum_wheel_joint
     name="back_left_joint"
@@ -248,5 +165,5 @@
     xyz="-0.03 -0.100 0"
     rpy="0 ${radians(270)} 0"
-    axis_z="-1"/>
+    axis_z="1"/>
   <xacro:mecanum_wheel_joint
     name="back_right_joint"
@@ -255,21 +172,4 @@
     xyz="0.03 -0.100 0"
     rpy="0 ${radians(90)} 0"
-    axis_z="1"/>
-  <!-- Attach mecanum rollers -->
-  <xacro:attach_mecanum_rollers
-    wheel_prefix="front_left"
-    wheel_link="front_left_wheel_1"
-    rot="-1"/>
-  <xacro:attach_mecanum_rollers
-    wheel_prefix="back_left"
-    wheel_link="back_left_wheel_1"
-    rot="1"/>
-  <xacro:attach_mecanum_rollers
-    wheel_prefix="front_right"
-    wheel_link="front_right_wheel_1"
-    rot="1"/>
-  <xacro:attach_mecanum_rollers
-    wheel_prefix="back_right"
-    wheel_link="back_right_wheel_1"
-    rot="-1"/>
+    axis_z="-1"/>
 </robot>

File: mecanumrover3_ros2/mecanumrover_description/urdf/mecanum3_ros2_control.xacro (robot description, xacro)
@@ -5,72 +5,24 @@
       <plugin>gazebo_ros2_control/GazeboSystem</plugin>
     </hardware>
-    <!-- Wheel joints (velocity)
-         min/max are required: GazeboSystem reads command_interface.max as fmax for the ODE
-         joint motor. Without them fmax=NaN→0 and the motor applies zero torque. -->
+    <!-- Wheel joints: STATE interfaces only (no command interface).
+         libgazebo_ros_diff_drive.so controls these joints directly via the Gazebo
+         physics API. If a velocity command_interface were present here, GazeboSystem
+         would initialise it to 0 and fight the diff_drive plugin. -->
     <joint name="front_left_joint">
-      <command_interface name="velocity">
-        <param name="min">-20.0</param>
-        <param name="max">20.0</param>
-      </command_interface>
-      <state_interface name="velocity"/>
-      <state_interface name="position"/>
-    </joint>
-    <joint name="front_right_joint">
-      <command_interface name="velocity">
-        <param name="min">-20.0</param>
-        <param name="max">20.0</param>
-      </command_interface>
-      <state_interface name="velocity"/>
-      <state_interface name="position"/>
-    </joint>
-    <joint name="back_left_joint">
-      <command_interface name="velocity">
-        <param name="min">-20.0</param>
-        <param name="max">20.0</param>
-      </command_interface>
-      <state_interface name="velocity"/>
-      <state_interface name="position"/>
-    </joint>
-    <joint name="back_right_joint">
-      <command_interface name="velocity">
-        <param name="min">-20.0</param>
-        <param name="max">20.0</param>
-      </command_interface>
-      <state_interface name="velocity"/>
-      <state_interface name="position"/>
-    </joint>
-    <!-- Gazebo internal spring/damping            -->
-    <joint name="front_left_suspension_joint">
       <state_interface name="position"/>
       <state_interface name="velocity"/>
     </joint>
-    <joint name="front_right_suspension_joint">
+    <joint name="front_right_joint">
       <state_interface name="position"/>
       <state_interface name="velocity"/>
     </joint>
-    <joint name="back_left_suspension_joint">
+    <joint name="back_left_joint">
       <state_interface name="position"/>
       <state_interface name="velocity"/>
     </joint>
-    <joint name="back_right_suspension_joint">
+    <joint name="back_right_joint">
       <state_interface name="position"/>
       <state_interface name="velocity"/>
     </joint>
-    <!-- Barrel joints (TF only, no control)       -->
-    <xacro:macro name="add_barrel_joints_recursive" params="prefix idx max_idx">
-      <joint name="${prefix}_barrel_${idx}_joint">
-        <state_interface name="position"/>
-      </joint>
-      <xacro:if value="${idx &lt; max_idx}">
-        <xacro:add_barrel_joints_recursive prefix="${prefix}" idx="${idx + 1}" max_idx="${max_idx}"/>
-      </xacro:if>
-    </xacro:macro>
-    <xacro:macro name="add_barrel_joints" params="prefix">
-      <xacro:add_barrel_joints_recursive prefix="${prefix}" idx="0" max_idx="14"/>
-    </xacro:macro>
-    <xacro:add_barrel_joints prefix="front_left"/>
-    <xacro:add_barrel_joints prefix="front_right"/>
-    <xacro:add_barrel_joints prefix="back_left"/>
-    <xacro:add_barrel_joints prefix="back_right"/>
   </ros2_control>
 </robot>
