Commit message: moveit2など

File: amir740_ros/amir_description/urdf/amir_for_rover.xacro (robot description, xacro)
@@ -3,4 +3,5 @@
 <xacro:include filename="$(find amir_description)/urdf/materials.xacro" />
 <xacro:include filename="$(find amir_description)/urdf/amir.trans" />
+<xacro:include filename="$(find vs_rover_options_description)/urdf/depth_cam/_d435.urdf.xacro" />
 <!-- <xacro:include filename="$(find amir_description)/urdf/amir.gazebo" />新しいros2用のやつを作る -->
 <!-- <xacro:include filename="$(find amir_description)/urdf/amir_mecanum3.gazebo.xacro" />
@@ -490,3 +491,7 @@
 </joint> -->
 <!-- end of outer joint -->
+<!-- D435 depth camera mounted at end effector (tcp_link) -->
+<xacro:sensor_d435 parent="tcp_link" name="d435" topics_ns="d435" use_nominal_extrinsics="true">
+  <origin xyz="0 -0.06 0.03" rpy="0 0 1.5708"/>
+</xacro:sensor_d435>
 </robot>

File: vs_rover_options_description/urdf/depth_cam/_d435.gazebo.xacro (robot description, xacro)
@@ -3,47 +3,14 @@
 License: Apache 2.0. See LICENSE file in root directory.
 Copyright(c) 2017 PAL Robotics, S.L. All Rights Reserved
-This is the Gazebo URDF model for the Intel RealSense D435 camera
+Ignition Gazebo (gz-sim 6 / Fortress) version.
+librealsense_gazebo_plugin / libgazebo_ros_camera は Classic 専用のため使用不可。
+ignition-gazebo-sensors-system (world SDF に登録済み) が rgbd_camera を処理し、
+ros_gz_bridge で ROS2 トピックへ変換する。
 -->
 <robot xmlns:xacro="http://ros.org/wiki/xacro">
   <xacro:macro name="gazebo_d435" params="camera_name reference_link topics_ns depth_optical_frame color_optical_frame infrared1_optical_frame infrared2_optical_frame publish_pointcloud:=true">
-    <!-- Load parameters to model's main link-->
-    <xacro:property name="deg_to_rad" value="0.01745329251994329577" />
     <gazebo reference="${reference_link}">
-      <self_collide>0</self_collide>
-      <enable_wind>0</enable_wind>
-      <kinematic>0</kinematic>
-      <gravity>1</gravity>
-      <!--<mu>1</mu>-->
-      <mu2>1</mu2>
-      <fdir1>0 0 0</fdir1>
-      <!--<slip1>0</slip1>
-      <slip2>0</slip2>-->
-      <kp>1e+13</kp>
-      <kd>1</kd>
-      <!--<max_vel>0.01</max_vel>
-      <min_depth>0</min_depth>-->
-      <sensor name="${camera_name}depth" type="depth">
-        <camera name="${camera_name}">
-          <horizontal_fov>1.57</horizontal_fov>
-          <image>
-            <width>1280</width>
-            <height>720</height>
-          </image>
-          <clip>
-            <near>0.1</near>
-            <far>100</far>
-          </clip>
-          <noise>
-            <type>gaussian</type>
-            <mean>0.0</mean>
-            <stddev>0.100</stddev>
-          </noise>
-        </camera>
-        <always_on>1</always_on>
-        <update_rate>30</update_rate>
-        <visualize>0</visualize>
-      </sensor>
-      <sensor name="${camera_name}color" type="camera">
-        <camera name="${camera_name}">
+      <sensor name="${camera_name}" type="rgbd_camera">
+        <camera>
           <horizontal_fov>1.57</horizontal_fov>
           <image>
@@ -54,6 +21,12 @@
           <clip>
             <near>0.1</near>
-            <far>100</far>
+            <far>100.0</far>
           </clip>
+          <depth_camera>
+            <clip>
+              <near>0.3</near>
+              <far>3.0</far>
+            </clip>
+          </depth_camera>
           <noise>
             <type>gaussian</type>
@@ -62,77 +35,10 @@
           </noise>
         </camera>
-        <always_on>1</always_on>
+        <always_on>true</always_on>
         <update_rate>30</update_rate>
-        <visualize>1</visualize>
+        <visualize>true</visualize>
+        <topic>${topics_ns}</topic>
+        <ignition_frame_id>${depth_optical_frame}</ignition_frame_id>
       </sensor>
-      <sensor name="${camera_name}ired1" type="camera">
-        <camera name="${camera_name}">
-          <horizontal_fov>1.57</horizontal_fov>
-          <image>
-            <width>1280</width>
-            <height>720</height>
-            <format>L_INT8</format>
-          </image>
-          <clip>
-            <near>0.1</near>
-            <far>100</far>
-          </clip>
-          <noise>
-            <type>gaussian</type>
-            <mean>0.0</mean>
-            <stddev>0.05</stddev>
-          </noise>
-        </camera>
-        <always_on>1</always_on>
-        <update_rate>1</update_rate>
-        <visualize>0</visualize>
-      </sensor>
-      <sensor name="${camera_name}ired2" type="camera">
-        <camera name="${camera_name}">
-          <horizontal_fov>1.57</horizontal_fov>
-          <image>
-            <width>1280</width>
-            <height>720</height>
-            <format>L_INT8</format>
-          </image>
-          <clip>
-            <near>0.1</near>
-            <far>100</far>
-          </clip>
-          <noise>
-            <type>gaussian</type>
-            <mean>0.0</mean>
-            <stddev>0.05</stddev>
-          </noise>
-        </camera>
-        <always_on>1</always_on>
-        <update_rate>1</update_rate>
-        <visualize>0</visualize>
-      </sensor>
-    </gazebo>
-    <gazebo>
-      <plugin name="${topics_ns}" filename="librealsense_gazebo_plugin.so">
-        <prefix>${camera_name}</prefix>
-        <depthUpdateRate>30.0</depthUpdateRate>
-        <colorUpdateRate>30.0</colorUpdateRate>
-        <infraredUpdateRate>1.0</infraredUpdateRate>
-        <depthTopicName>depth/image_raw</depthTopicName>
-        <depthCameraInfoTopicName>depth/camera_info</depthCameraInfoTopicName>
-        <colorTopicName>color/image_raw</colorTopicName>
-        <colorCameraInfoTopicName>color/camera_info</colorCameraInfoTopicName>
-        <infrared1TopicName>infra1/image_raw</infrared1TopicName>
-        <infrared1CameraInfoTopicName>infra1/camera_info</infrared1CameraInfoTopicName>
-        <infrared2TopicName>infra2/image_raw</infrared2TopicName>
-        <infrared2CameraInfoTopicName>infra2/camera_info</infrared2CameraInfoTopicName>
-        <colorOpticalframeName>${color_optical_frame}</colorOpticalframeName>
-        <depthOpticalframeName>${depth_optical_frame}</depthOpticalframeName>
-        <infrared1OpticalframeName>${infrared1_optical_frame}</infrared1OpticalframeName>
-        <infrared2OpticalframeName>${infrared2_optical_frame}</infrared2OpticalframeName>
-        <rangeMinDepth>0.3</rangeMinDepth>
-        <rangeMaxDepth>3.0</rangeMaxDepth>
-        <pointCloud>true</pointCloud>
-        <pointCloudTopicName>depth/color/points</pointCloudTopicName>
-        <pointCloudCutoff>0.3</pointCloudCutoff>
-      </plugin>
     </gazebo>
   </xacro:macro>

File: vs_rover_options_description/urdf/depth_cam/_d435.urdf.xacro (robot description, xacro)
@@ -75,4 +75,12 @@
       </inertial>
     </link>
+    <!-- Ignition Gazebo (Ogre2) は DAE の Lambert マテリアルを自動適用しないため明示する -->
+    <gazebo reference="${name}_link">
+      <material>
+        <ambient>0.39 0.39 0.39 1</ambient>
+        <diffuse>0.39 0.39 0.39 1</diffuse>
+        <specular>0.1 0.1 0.1 1</specular>
+      </material>
+    </gazebo>
     <!-- Use the nominal extrinsics between camera frames if the calibrated extrinsics aren't being published. e.g. running the device in simulation  -->
     <xacro:if value="${use_nominal_extrinsics}">

File: vs_rover_options_description/urdf/lrf/tg30_mecanum3.xacro (robot description, xacro)
@@ -1,3 +1,5 @@
 <robot name="lrf_tg30_mecanum3" xmlns:xacro="http://ros.org/wiki/xacro">
+  <!-- 後部 LRF を有効にする場合は use_back_lrf:=true を渡す -->
+  <xacro:arg name="use_back_lrf" default="false" />
   <xacro:include filename="$(find vs_rover_options_description)/urdf/lrf/tg30_mecanum3.gazebo" />
   <xacro:property name="tg30_lrf_front_x_offset" value="0.0" />
@@ -37,4 +39,6 @@
     </collision>
   </link>
+  <!-- 後部 LRF: use_back_lrf:=true で復活 (デフォルト false = 無効) -->
+  <xacro:if value="$(arg use_back_lrf)">
   <joint name="back_lrf_joint" type="fixed">
     <parent link="base_link" />
@@ -64,3 +68,4 @@
     </collision>
   </link>
+  </xacro:if>
 </robot>

Commit message: gz軽く

File: amir740_ros/amir_description/urdf/amir_for_rover.xacro (robot description, xacro)
@@ -26,7 +26,7 @@
   </visual>
   <collision>
-    <origin xyz="0 0 0" rpy="0 0 0"/>
-    <geometry>
-      <mesh filename="package://amir_description/meshes/base_link.stl" scale="0.001 0.001 0.001"/>
+    <origin xyz="0 0 -0.165" rpy="0 0 0"/>
+    <geometry>
+      <box size="0.15 0.12 0.33"/>
     </geometry>
   </collision>
@@ -51,7 +51,7 @@
   </visual>
   <collision>
-    <origin xyz="0.00 0.001523 0.097" rpy="0 0 0"/>
-    <geometry>
-      <mesh filename="package://amir_description/meshes/link1_1.stl" scale="0.001 0.001 0.001"/>
+    <origin xyz="0 0.001523 0.048" rpy="0 0 0"/>
+    <geometry>
+      <cylinder radius="0.055" length="0.10"/>
     </geometry>
   </collision>
@@ -76,7 +76,7 @@
   </visual>
   <collision>
-    <origin xyz="0.0 0.001523 -0.0" rpy="0 0 0"/>
-    <geometry>
-      <mesh filename="package://amir_description/meshes/link2_1.stl" scale="0.001 0.001 0.001"/>
+    <origin xyz="0 0.155 0" rpy="1.5708 0 0"/>
+    <geometry>
+      <cylinder radius="0.045" length="0.31"/>
     </geometry>
   </collision>
@@ -101,7 +101,7 @@
   </visual>
   <collision>
-    <origin xyz="-0.0 -0.308477 0.0" rpy="0 0 0"/>
-    <geometry>
-      <mesh filename="package://amir_description/meshes/link3_1.stl" scale="0.001 0.001 0.001"/>
+    <origin xyz="0 0.155 0" rpy="1.5708 0 0"/>
+    <geometry>
+      <cylinder radius="0.040" length="0.31"/>
     </geometry>
   </collision>
@@ -126,7 +126,7 @@
   </visual>
   <collision>
-    <origin xyz="0.0 -0.618477 -0.0" rpy="0 0 0"/>
-    <geometry>
-      <mesh filename="package://amir_description/meshes/link4_1.stl" scale="0.001 0.001 0.001"/>
+    <origin xyz="0 0.020 0" rpy="0 0 0"/>
+    <geometry>
+      <box size="0.065 0.042 0.060"/>
     </geometry>
   </collision>

File: amir740_ros/amir_description/urdf/amir_mecanum3_sim.xacro (robot description, xacro)
@@ -162,5 +162,5 @@
           <ode>
             <kp>1e6</kp>
-            <kd>1e3</kd>
+            <kd>1e2</kd>
             <max_vel>0.01</max_vel>
             <min_depth>0.001</min_depth>
@@ -182,5 +182,5 @@
           <ode>
             <kp>1e6</kp>
-            <kd>1e3</kd>
+            <kd>1e2</kd>
             <max_vel>0.01</max_vel>
             <min_depth>0.001</min_depth>
