Commit message: gazebo222

File: mecanumrover3_ros2/mecanumrover_description/urdf/mecanum3.xacro (robot description, xacro)
@@ -185,4 +185,9 @@
       <origin xyz="${xyz}" rpy="${rpy}"/>
       <axis xyz="0 0 ${axis_z}"/>
+      <!-- effort limit is required: GazeboSystem uses it as ODE fmax.
+           Without it fmax=0 and the velocity controller applies zero torque,
+           letting reaction forces from the arm push the base freely. -->
+      <limit effort="50.0" velocity="20.0"/>
+      <dynamics damping="1.0" friction="0.0"/>
     </joint>
   </xacro:macro>

Commit message: madamondaiari

File: mecanumrover3_ros2/mecanumrover_description/urdf/mecanum3.xacro (robot description, xacro)
@@ -25,5 +25,5 @@
         rpy="${pi/4*rot} 0 ${radians(dir)}"/>
       <axis xyz="0 0 1"/>
-      <dynamics damping="0.001" friction="0.0"/>
+      <dynamics damping="0.001" friction="0.001"/>
     </joint>
     <link name="${prefix}_link">
@@ -80,5 +80,5 @@
     <inertial>
       <origin xyz="0.000129 -0.001817 0.110883"/>
-      <mass value="14"/>
+      <mass value="40"/>
       <inertia ixx="1.346868e-01" iyy="4.468661e-02" izz="1.499091e-01" ixy="3.076527e-04" ixz="-2.931603e-05" iyz="2.763693e-05"/>
     </inertial>
@@ -188,5 +188,5 @@
            Without it fmax=0 and the velocity controller applies zero torque,
            letting reaction forces from the arm push the base freely. -->
-      <limit effort="50.0" velocity="20.0"/>
+      <limit effort="1500.0" velocity="20.0"/>
       <dynamics damping="1.0" friction="0.0"/>
     </joint>

File: mecanumrover3_ros2/mecanumrover_description/urdf/mecanum3_ros2_control.xacro (robot description, xacro)
@@ -5,22 +5,36 @@
       <plugin>gazebo_ros2_control/GazeboSystem</plugin>
     </hardware>
-    <!-- Wheel joints (velocity) -->
+    <!-- Wheel joints (velocity)
+         min/max are required: GazeboSystem reads command_interface.max as fmax for the ODE
+         joint motor. Without them fmax=NaN→0 and the motor applies zero torque. -->
     <joint name="front_left_joint">
-      <command_interface name="velocity"/>
+      <command_interface name="velocity">
+        <param name="min">-20.0</param>
+        <param name="max">20.0</param>
+      </command_interface>
       <state_interface name="velocity"/>
       <state_interface name="position"/>
     </joint>
     <joint name="front_right_joint">
-      <command_interface name="velocity"/>
+      <command_interface name="velocity">
+        <param name="min">-20.0</param>
+        <param name="max">20.0</param>
+      </command_interface>
       <state_interface name="velocity"/>
       <state_interface name="position"/>
     </joint>
     <joint name="back_left_joint">
-      <command_interface name="velocity"/>
+      <command_interface name="velocity">
+        <param name="min">-20.0</param>
+        <param name="max">20.0</param>
+      </command_interface>
       <state_interface name="velocity"/>
       <state_interface name="position"/>
     </joint>
     <joint name="back_right_joint">
-      <command_interface name="velocity"/>
+      <command_interface name="velocity">
+        <param name="min">-20.0</param>
+        <param name="max">20.0</param>
+      </command_interface>
       <state_interface name="velocity"/>
       <state_interface name="position"/>

Commit message: nav2と把持できたﾆｮ

File: mecanumrover3_ros2/mecanumrover_description/urdf/mecanum3.xacro (robot description, xacro)
@@ -5,4 +5,68 @@
   <xacro:include filename="$(find mecanumrover_description)/urdf/mecanum3_ros2_control.xacro" />
   <xacro:include filename="$(find vs_rover_options_description)/urdf/lrf/tg30_mecanum3.xacro" />
+  <!-- Inertial macros -->
+  <xacro:macro name="cylinder_inertial" params="mass radius length">
+    <mass value="${mass}"/>
+    <inertia
+      ixx="${((radius*radius)/4 + (length*length)/12)*mass}"
+      ixy="0" ixz="0"
+      iyy="${((radius*radius)/4 + (length*length)/12)*mass}"
+      iyz="0"
+      izz="${(mass*radius*radius)/2}" />
+  </xacro:macro>
+  <!-- Barrel (roller) macros -->
+  <xacro:macro name="barrel_rl" params="prefix parent dir rot">
+    <joint name="${prefix}_joint" type="continuous">
+      <parent link="${parent}"/>
+      <child  link="${prefix}_link"/>
+      <origin
+        xyz="${0.0666389*cos(radians(dir))} ${0.0666389*sin(radians(dir))} 0"
+        rpy="${pi/4*rot} 0 ${radians(dir)}"/>
+      <axis xyz="0 0 1"/>
+      <dynamics damping="0.001" friction="0.0"/>
+    </joint>
+    <link name="${prefix}_link">
+      <visual>
+        <geometry>
+          <mesh filename="package://mecanumrover_description/meshes/mecanum3/mecanum_barrel.stl"/>
+        </geometry>
+        <material name="dark_grey"/>
+      </visual>
+      <collision>
+        <geometry>
+          <mesh filename="package://mecanumrover_description/meshes/mecanum3/mecanum_barrel.stl"/>
+        </geometry>
+      </collision>
+      <inertial>
+        <xacro:cylinder_inertial
+          mass="0.01225"
+          radius="0.00956"
+          length="0.0381"/>
+      </inertial>
+    </link>
+  </xacro:macro>
+  <xacro:macro name="barrels_rl" params="prefix parent rot">
+    <xacro:barrel_rl prefix="${prefix}_0"  parent="${parent}" dir="0"   rot="${rot}"/>
+    <xacro:barrel_rl prefix="${prefix}_1"  parent="${parent}" dir="24"  rot="${rot}"/>
+    <xacro:barrel_rl prefix="${prefix}_2"  parent="${parent}" dir="48"  rot="${rot}"/>
+    <xacro:barrel_rl prefix="${prefix}_3"  parent="${parent}" dir="72"  rot="${rot}"/>
+    <xacro:barrel_rl prefix="${prefix}_4"  parent="${parent}" dir="96"  rot="${rot}"/>
+    <xacro:barrel_rl prefix="${prefix}_5"  parent="${parent}" dir="120" rot="${rot}"/>
+    <xacro:barrel_rl prefix="${prefix}_6"  parent="${parent}" dir="144" rot="${rot}"/>
+    <xacro:barrel_rl prefix="${prefix}_7"  parent="${parent}" dir="168" rot="${rot}"/>
+    <xacro:barrel_rl prefix="${prefix}_8"  parent="${parent}" dir="192" rot="${rot}"/>
+    <xacro:barrel_rl prefix="${prefix}_9"  parent="${parent}" dir="216" rot="${rot}"/>
+    <xacro:barrel_rl prefix="${prefix}_10" parent="${parent}" dir="240" rot="${rot}"/>
+    <xacro:barrel_rl prefix="${prefix}_11" parent="${parent}" dir="264" rot="${rot}"/>
+    <xacro:barrel_rl prefix="${prefix}_12" parent="${parent}" dir="288" rot="${rot}"/>
+    <xacro:barrel_rl prefix="${prefix}_13" parent="${parent}" dir="312" rot="${rot}"/>
+    <xacro:barrel_rl prefix="${prefix}_14" parent="${parent}" dir="336" rot="${rot}"/>
+  </xacro:macro>
+  <xacro:macro name="attach_mecanum_rollers" params="wheel_prefix wheel_link rot">
+    <xacro:barrels_rl
+      prefix="${wheel_prefix}_barrel"
+      parent="${wheel_link}"
+      rot="${rot}"/>
+  </xacro:macro>
   <!-- Arm link macro -->
   <xacro:macro name="mecanum_arm_link" params="name">
@@ -29,6 +93,6 @@
   </xacro:macro>
   <!-- Wheel link macros
-       Collision changed from mecanum STL mesh to cylinder for stable ODE contact.
-       radius=0.076 matches the mecanum outer radius (barrel center 0.0666 + barrel radius 0.00956). -->
+       Collision uses the actual STL mesh so barrel rollers are the outermost
+       contact geometry (no separate cylinder approximation needed). -->
   <xacro:macro name="mecanum_wheel_link" params="name">
     <link name="${name}">
@@ -47,5 +111,6 @@
       <collision>
         <geometry>
-          <cylinder radius="0.076" length="0.05"/>
+          <mesh filename="package://mecanumrover_description/meshes/mecanum3/mecanum_wheel.stl"
+                scale="0.001 0.001 0.001"/>
         </geometry>
       </collision>
@@ -68,5 +133,6 @@
       <collision>
         <geometry>
-          <cylinder radius="0.076" length="0.05"/>
+          <mesh filename="package://mecanumrover_description/meshes/mecanum3/mecanum_wheel_rev.stl"
+                scale="0.001 0.001 0.001"/>
         </geometry>
       </collision>
@@ -174,3 +240,22 @@
     rpy="0 ${radians(90)} 0"
     axis_z="-1"/>
+  <!-- Attach mecanum rollers (15 barrels per wheel at 24° intervals, ±45° tilt)
+       rot=-1 → -45° tilt (rev wheel pattern: front_left, back_right)
+       rot=+1 → +45° tilt (normal wheel pattern: front_right, back_left) -->
+  <xacro:attach_mecanum_rollers
+    wheel_prefix="front_left"
+    wheel_link="front_left_wheel_1"
+    rot="-1"/>
+  <xacro:attach_mecanum_rollers
+    wheel_prefix="front_right"
+    wheel_link="front_right_wheel_1"
+    rot="1"/>
+  <xacro:attach_mecanum_rollers
+    wheel_prefix="back_left"
+    wheel_link="back_left_wheel_1"
+    rot="1"/>
+  <xacro:attach_mecanum_rollers
+    wheel_prefix="back_right"
+    wheel_link="back_right_wheel_1"
+    rot="-1"/>
 </robot>

File: mecanumrover3_ros2/mecanumrover_description/urdf/mecanum3_ros2_control.xacro (robot description, xacro)
@@ -3,5 +3,5 @@
   <ros2_control name="MecanumSystem" type="system">
     <hardware>
-      <!-- Ignition Gazebo hardware plugin (replaces gazebo_ros2_control/GazeboSystem) -->
+      <!-- Ignition Gazebo hardware plugin (matches gz_ros2_control-system in mecanum3.gazebo) -->
       <plugin>gz_ros2_control/GazeboSimSystem</plugin>
     </hardware>

Commit message: light

File: mecanumrover3_ros2/mecanumrover_description/urdf/mecanum3.xacro (robot description, xacro)
@@ -4,69 +4,6 @@
   <xacro:include filename="$(find mecanumrover_description)/urdf/mecanum3.gazebo" />
   <xacro:include filename="$(find mecanumrover_description)/urdf/mecanum3_ros2_control.xacro" />
+  <!-- OPTION: LRF TG30 -->
   <xacro:include filename="$(find vs_rover_options_description)/urdf/lrf/tg30_mecanum3.xacro" />
-  <!-- Inertial macros -->
-  <xacro:macro name="cylinder_inertial" params="mass radius length">
-    <mass value="${mass}"/>
-    <inertia
-      ixx="${((radius*radius)/4 + (length*length)/12)*mass}"
-      ixy="0" ixz="0"
-      iyy="${((radius*radius)/4 + (length*length)/12)*mass}"
-      iyz="0"
-      izz="${(mass*radius*radius)/2}" />
-  </xacro:macro>
-  <!-- Barrel (roller) macros -->
-  <xacro:macro name="barrel_rl" params="prefix parent dir rot">
-    <joint name="${prefix}_joint" type="continuous">
-      <parent link="${parent}"/>
-      <child  link="${prefix}_link"/>
-      <origin
-        xyz="${0.0666389*cos(radians(dir))} ${0.0666389*sin(radians(dir))} 0"
-        rpy="${pi/4*rot} 0 ${radians(dir)}"/>
-      <axis xyz="0 0 1"/>
-      <dynamics damping="0.001" friction="0.0"/>
-    </joint>
-    <link name="${prefix}_link">
-      <visual>
-        <geometry>
-          <mesh filename="package://mecanumrover_description/meshes/mecanum3/mecanum_barrel.stl"/>
-        </geometry>
-        <material name="dark_grey"/>
-      </visual>
-      <collision>
-        <geometry>
-          <mesh filename="package://mecanumrover_description/meshes/mecanum3/mecanum_barrel.stl"/>
-        </geometry>
-      </collision>
-      <inertial>
-        <xacro:cylinder_inertial
-          mass="0.01225"
-          radius="0.00956"
-          length="0.0381"/>
-      </inertial>
-    </link>
-  </xacro:macro>
-  <xacro:macro name="barrels_rl" params="prefix parent rot">
-    <xacro:barrel_rl prefix="${prefix}_0"  parent="${parent}" dir="0"   rot="${rot}"/>
-    <xacro:barrel_rl prefix="${prefix}_1"  parent="${parent}" dir="24"  rot="${rot}"/>
-    <xacro:barrel_rl prefix="${prefix}_2"  parent="${parent}" dir="48"  rot="${rot}"/>
-    <xacro:barrel_rl prefix="${prefix}_3"  parent="${parent}" dir="72"  rot="${rot}"/>
-    <xacro:barrel_rl prefix="${prefix}_4"  parent="${parent}" dir="96"  rot="${rot}"/>
-    <xacro:barrel_rl prefix="${prefix}_5"  parent="${parent}" dir="120" rot="${rot}"/>
-    <xacro:barrel_rl prefix="${prefix}_6"  parent="${parent}" dir="144" rot="${rot}"/>
-    <xacro:barrel_rl prefix="${prefix}_7"  parent="${parent}" dir="168" rot="${rot}"/>
-    <xacro:barrel_rl prefix="${prefix}_8"  parent="${parent}" dir="192" rot="${rot}"/>
-    <xacro:barrel_rl prefix="${prefix}_9"  parent="${parent}" dir="216" rot="${rot}"/>
-    <xacro:barrel_rl prefix="${prefix}_10" parent="${parent}" dir="240" rot="${rot}"/>
-    <xacro:barrel_rl prefix="${prefix}_11" parent="${parent}" dir="264" rot="${rot}"/>
-    <xacro:barrel_rl prefix="${prefix}_12" parent="${parent}" dir="288" rot="${rot}"/>
-    <xacro:barrel_rl prefix="${prefix}_13" parent="${parent}" dir="312" rot="${rot}"/>
-    <xacro:barrel_rl prefix="${prefix}_14" parent="${parent}" dir="336" rot="${rot}"/>
-  </xacro:macro>
-  <xacro:macro name="attach_mecanum_rollers" params="wheel_prefix wheel_link rot">
-    <xacro:barrels_rl
-      prefix="${wheel_prefix}_barrel"
-      parent="${wheel_link}"
-      rot="${rot}"/>
-  </xacro:macro>
   <!-- Arm link macro -->
   <xacro:macro name="mecanum_arm_link" params="name">
@@ -92,7 +29,5 @@
     </link>
   </xacro:macro>
-  <!-- Wheel link macros
-       Collision uses the actual STL mesh so barrel rollers are the outermost
-       contact geometry (no separate cylinder approximation needed). -->
+  <!-- Wheel link macros (cylinder collision for simple differential drive physics) -->
   <xacro:macro name="mecanum_wheel_link" params="name">
     <link name="${name}">
@@ -111,6 +46,5 @@
       <collision>
         <geometry>
-          <mesh filename="package://mecanumrover_description/meshes/mecanum3/mecanum_wheel.stl"
-                scale="0.001 0.001 0.001"/>
+          <cylinder radius="0.076" length="0.044"/>
         </geometry>
       </collision>
@@ -120,5 +54,5 @@
     <link name="${name}">
       <inertial>
-        <origin xyz="0.000657 0 0.007742"/>
+        <origin xyz="0 0 0"/>
         <mass value="0.88"/>
         <inertia ixx="7.655818e-04" iyy="7.655769e-04" izz="8.900386e-04" ixy="-6.106217e-09" ixz="1.064093e-09" iyz="-2.991811e-09"/>
@@ -133,6 +67,5 @@
       <collision>
         <geometry>
-          <mesh filename="package://mecanumrover_description/meshes/mecanum3/mecanum_wheel_rev.stl"
-                scale="0.001 0.001 0.001"/>
+          <cylinder radius="0.076" length="0.044"/>
         </geometry>
       </collision>
@@ -240,22 +173,3 @@
     rpy="0 ${radians(90)} 0"
     axis_z="-1"/>
-  <!-- Attach mecanum rollers (15 barrels per wheel at 24° intervals, ±45° tilt)
-       rot=-1 → -45° tilt (rev wheel pattern: front_left, back_right)
-       rot=+1 → +45° tilt (normal wheel pattern: front_right, back_left) -->
-  <xacro:attach_mecanum_rollers
-    wheel_prefix="front_left"
-    wheel_link="front_left_wheel_1"
-    rot="-1"/>
-  <xacro:attach_mecanum_rollers
-    wheel_prefix="front_right"
-    wheel_link="front_right_wheel_1"
-    rot="1"/>
-  <xacro:attach_mecanum_rollers
-    wheel_prefix="back_left"
-    wheel_link="back_left_wheel_1"
-    rot="1"/>
-  <xacro:attach_mecanum_rollers
-    wheel_prefix="back_right"
-    wheel_link="back_right_wheel_1"
-    rot="-1"/>
 </robot>

File: mecanumrover3_ros2/mecanumrover_description/urdf/mecanum3_ros2_control.xacro (robot description, xacro)
@@ -3,10 +3,8 @@
   <ros2_control name="MecanumSystem" type="system">
     <hardware>
-      <!-- Ignition Gazebo hardware plugin (matches gz_ros2_control-system in mecanum3.gazebo) -->
+      <!-- Ignition Gazebo hardware plugin -->
       <plugin>gz_ros2_control/GazeboSimSystem</plugin>
     </hardware>
-    <!-- Wheel joints: velocity COMMAND interfaces required by mecanum_drive_controller.
-         Classic Gazebo used libgazebo_ros_diff_drive.so which bypassed ros2_control.
-         In Ignition, mecanum_drive_controller drives the wheels via these interfaces. -->
+    <!-- Wheel joints: velocity COMMAND interfaces for mecanum_drive_controller -->
     <joint name="front_left_joint">
       <command_interface name="velocity">
